Commit message: Changed location of the lidar

File: gazebo/macros.xacro (robot description, xacro)
@@ -227,5 +227,5 @@
     <joint name="rplidar_joint" type="fixed">
       <axis xyz="0 1 0" />
-      <origin xyz="0.02 0 0.058" rpy="0 0 3.14"/>
+      <origin xyz="0.02 0 0" rpy="0 0 3.14"/>
       <parent link="base_link"/>
       <child link="laser"/>
